Commit message: add ORCA meshes

File: roto/assets/orca/models/urdf/orcahand_right.urdf (robot description, URDF)
Before this commit: robot orcahand_right, 42 links, 41 joints
Links:
- link right_index_ip: geometry collision mesh filename=package://orcahand_description/assets/urdf/right/collision/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; collision mesh filename=package://orcahand_description/assets/urdf/right/collision/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
- link right_index_mp: geometry collision mesh filename=package://orcahand_description/assets/urdf/right/collision/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; visual mesh filename=package://orcahand_description/assets/urdf/right/visual/rig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
- link right_index_pp: geometry collision mesh filename=package://orcahand_description/assets/urdf/right/collision/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; collision mesh filename=package://orcahand_description/assets/urdf/right/collision/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
- link right_middle_ip: geometry collision mesh filename=package://orcahand_description/assets/urdf/right/collision/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; collision mesh filename=package://orcahand_description/assets/urdf/right/collision/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
- link right_middle_mp: geometry collision mesh filename=package://orcahand_description/assets/urdf/right/collision/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; visual mesh filename=package://orcahand_description/assets/urdf/right/visual/rig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
- link right_middle_pp: geometry collision mesh filename=package://orcahand_description/assets/urdf/right/collision/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; collision mesh filename=package://orcahand_description/assets/urdf/right/collision/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
- link right_palm: geometry collision mesh filename=package://orcahand_description/assets/urdf/right/collision/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; collision mesh filename=package://orcahand_description/assets/urdf/right/collision/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
- link right_pinky_ip: geometry collision mesh filename=package://orcahand_description/assets/urdf/right/collision/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; collision mesh filename=package://orcahand_description/assets/urdf/right/collision/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
- link right_pinky_mp: geometry collision mesh filename=package://orcahand_description/assets/urdf/right/collision/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; visual mesh filename=package://orcahand_description/assets/urdf/right/visual/rig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
- link right_pinky_pp: geometry collision mesh filename=package://orcahand_description/assets/urdf/right/collision/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; collision mesh filename=package://orcahand_description/assets/urdf/right/collision/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
- link right_ring_ip: geometry collision mesh filename=package://orcahand_description/assets/urdf/right/collision/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; collision mesh filename=package://orcahand_description/assets/urdf/right/collision/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
- link right_ring_mp: geometry collision mesh filename=package://orcahand_description/assets/urdf/right/collision/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; visual mesh filename=package://orcahand_description/assets/urdf/right/visual/rig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
- link right_ring_pp: geometry collision mesh filename=package://orcahand_description/assets/urdf/right/collision/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; collision mesh filename=package://orcahand_description/assets/urdf/right/collision/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
- link right_thumb_dp: geometry collision mesh filename=package://orcahand_description/assets/urdf/right/collision/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; collision mesh filename=package://orcahand_description/assets/urdf/right/collision/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
- link right_thumb_ip: geometry collision mesh filename=package://orcahand_description/assets/urdf/right/collision/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; collision mesh filename=package://orcahand_description/assets/urdf/right/collision/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
- link right_thumb_mp: geometry collision mesh filename=package://orcahand_description/assets/urdf/right/collision/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; visual mesh filename=package://orcahand_description/assets/urdf/right/visual/rig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
- link right_thumb_pp: geometry collision mesh filename=package://orcahand_description/assets/urdf/right/collision/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; visual mesh filename=package://orcahand_description/assets/urdf/right/visual/rig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
- link right_tower: geometry collision mesh filename=package://orcahand_description/assets/urdf/right/collision/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; collision mesh filename=package://orcahand_description/assets/urdf/right/collision/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
Joints:
- joint right_index_pip: limit lower=0.0 upper=1.88496 effort=100 velocity=100 -> lower=-0.34907 upper=1.88496 effort=100 velocity=100
- joint right_middle_pip: limit lower=0.0 upper=1.8675 effort=100 velocity=100 -> lower=-0.34907 upper=1.8675 effort=100 velocity=100
- joint right_pinky_pip: limit lower=0.0 upper=1.88496 effort=100 velocity=100 -> lower=-0.34907 upper=1.88496 effort=100 velocity=100
- joint right_ring_pip: limit lower=0.0 upper=1.8675 effort=100 velocity=100 -> lower=-0.34907 upper=1.8675 effort=100 velocity=100

File: roto/assets/orca/models/urdf/orcahand_right_extended.urdf (robot description, URDF)
Before this commit: robot orcahand_right, 42 links, 41 joints
Links:
- link right_index_ip: geometry collision mesh filename=package://orcahand_description/assets/urdf/right/collision/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; collision mesh filename=package://orcahand_description/assets/urdf/right/collision/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
- link right_index_mp: geometry collision mesh filename=package://orcahand_description/assets/urdf/right/collision/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; visual mesh filename=package://orcahand_description/assets/urdf/right/visual/rig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
- link right_index_pp: geometry collision mesh filename=package://orcahand_description/assets/urdf/right/collision/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; collision mesh filename=package://orcahand_description/assets/urdf/right/collision/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
- link right_middle_ip: geometry collision mesh filename=package://orcahand_description/assets/urdf/right/collision/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; collision mesh filename=package://orcahand_description/assets/urdf/right/collision/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
- link right_middle_mp: geometry collision mesh filename=package://orcahand_description/assets/urdf/right/collision/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; visual mesh filename=package://orcahand_description/assets/urdf/right/visual/rig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
- link right_middle_pp: geometry collision mesh filename=package://orcahand_description/assets/urdf/right/collision/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; collision mesh filename=package://orcahand_description/assets/urdf/right/collision/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
- link right_palm: geometry collision mesh filename=package://orcahand_description/assets/urdf/right/collision/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; collision mesh filename=package://orcahand_description/assets/urdf/right/collision/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
- link right_pinky_ip: geometry collision mesh filename=package://orcahand_description/assets/urdf/right/collision/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; collision mesh filename=package://orcahand_description/assets/urdf/right/collision/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
- link right_pinky_mp: geometry collision mesh filename=package://orcahand_description/assets/urdf/right/collision/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; visual mesh filename=package://orcahand_description/assets/urdf/right/visual/rig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
- link right_pinky_pp: geometry collision mesh filename=package://orcahand_description/assets/urdf/right/collision/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; collision mesh filename=package://orcahand_description/assets/urdf/right/collision/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
- link right_ring_ip: geometry collision mesh filename=package://orcahand_description/assets/urdf/right/collision/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; collision mesh filename=package://orcahand_description/assets/urdf/right/collision/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
- link right_ring_mp: geometry collision mesh filename=package://orcahand_description/assets/urdf/right/collision/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; visual mesh filename=package://orcahand_description/assets/urdf/right/visual/rig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
- link right_ring_pp: geometry collision mesh filename=package://orcahand_description/assets/urdf/right/collision/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; collision mesh filename=package://orcahand_description/assets/urdf/right/collision/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
- link right_thumb_dp: geometry collision mesh filename=package://orcahand_description/assets/urdf/right/collision/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; collision mesh filename=package://orcahand_description/assets/urdf/right/collision/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
- link right_thumb_ip: geometry collision mesh filename=package://orcahand_description/assets/urdf/right/collision/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; collision mesh filename=package://orcahand_description/assets/urdf/right/collision/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
- link right_thumb_mp: geometry collision mesh filename=package://orcahand_description/assets/urdf/right/collision/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; visual mesh filename=package://orcahand_description/assets/urdf/right/visual/rig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
- link right_thumb_pp: geometry collision mesh filename=package://orcahand_description/assets/urdf/right/collision/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; visual mesh filename=package://orcahand_description/assets/urdf/right/visual/rig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
- link right_tower: geometry collision mesh filename=package://orcahand_description/assets/urdf/right/collision/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; collision mesh filename=package://orcahand_description/assets/urdf/right/collision/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
Joints:
- joint right_index_pip: limit lower=0.0 upper=1.88496 effort=100 velocity=100 -> lower=-0.34907 upper=1.88496 effort=100 velocity=100
- joint right_middle_pip: limit lower=0.0 upper=1.8675 effort=100 velocity=100 -> lower=-0.34907 upper=1.8675 effort=100 velocity=100
- joint right_pinky_pip: limit lower=0.0 upper=1.88496 effort=100 velocity=100 -> lower=-0.34907 upper=1.88496 effort=100 velocity=100
- joint right_ring_pip: limit lower=0.0 upper=1.8675 effort=100 velocity=100 -> lower=-0.34907 upper=1.8675 effort=100 velocity=100
