Commit message: orca fixed urdf, articulationcfg, bounce ball pos

File: roto/assets/orca/orcahand_right.urdf (robot description, URDF)
Before this commit: robot orcahand_right, 42 links, 41 joints
Links:
- link right_index_ip: geometry collision mesh filename=meshes/urdf/right/collision/right_collision_index_ip_mesh.s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; collision mesh filename=meshes/urdf/right/collision/right_collision_index_ip_skin_m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
- link right_index_mp: geometry collision mesh filename=meshes/urdf/right/collision/right_collision_index_mp_mesh.s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; visual mesh filename=meshes/urdf/right/visual/right_visual_index_mp_mesh.stl
- link right_index_pp: geometry collision mesh filename=meshes/urdf/right/collision/right_collision_index_pp_mesh.s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; collision mesh filename=meshes/urdf/right/collision/right_collision_index_pp_skin_m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
- link right_middle_ip: geometry collision mesh filename=meshes/urdf/right/collision/right_collision_middle_ip_mesh.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; collision mesh filename=meshes/urdf/right/collision/right_collision_middle_ip_skin_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
- link right_middle_mp: geometry collision mesh filename=meshes/urdf/right/collision/right_collision_middle_mp_mesh.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; visual mesh filename=meshes/urdf/right/visual/right_visual_middle_mp_mesh.stl
- link right_middle_pp: geometry collision mesh filename=meshes/urdf/right/collision/right_collision_middle_pp_mesh.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; collision mesh filename=meshes/urdf/right/collision/right_collision_middle_pp_skin_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
- link right_palm: geometry collision mesh filename=meshes/urdf/right/collision/right_collision_palm_mesh.stl; collision mesh filename=meshes/urdf/right/collision/right_collision_palm_skin_mesh.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
- link right_pinky_ip: geometry collision mesh filename=meshes/urdf/right/collision/right_collision_pinky_ip_mesh.s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; collision mesh filename=meshes/urdf/right/collision/right_collision_pinky_ip_skin_m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
- link right_pinky_mp: geometry collision mesh filename=meshes/urdf/right/collision/right_collision_pinky_mp_mesh.s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; visual mesh filename=meshes/urdf/right/visual/right_visual_pinky_mp_mesh.stl
- link right_pinky_pp: geometry collision mesh filename=meshes/urdf/right/collision/right_collision_pinky_pp_mesh.s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; collision mesh filename=meshes/urdf/right/collision/right_collision_pinky_pp_skin_m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
- link right_ring_ip: geometry collision mesh filename=meshes/urdf/right/collision/right_collision_ring_ip_mesh.stl; collision mesh filename=meshes/urdf/right/collision/right_collision_ring_ip_skin_me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
- link right_ring_mp: geometry collision mesh filename=meshes/urdf/right/collision/right_collision_ring_mp_mesh.stl; visual mesh filename=meshes/urdf/right/visual/right_visual_ring_mp_mesh.stl
- link right_ring_pp: geometry collision mesh filename=meshes/urdf/right/collision/right_collision_ring_pp_mesh.stl; collision mesh filename=meshes/urdf/right/collision/right_collision_ring_pp_skin_me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
- link right_thumb_dp: geometry collision mesh filename=meshes/urdf/right/collision/right_collision_thumb_dp_mesh.s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; collision mesh filename=meshes/urdf/right/collision/right_collision_thumb_dp_skin_m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
- link right_thumb_ip: geometry collision mesh filename=meshes/urdf/right/collision/right_collision_thumb_ip_mesh.s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; collision mesh filename=meshes/urdf/right/collision/right_collision_thumb_ip_skin_m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
- link right_thumb_mp: geometry collision mesh filename=meshes/urdf/right/collision/right_collision_thumb_mp_mesh.s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; visual mesh filename=meshes/urdf/right/visual/right_visual_thumb_mp_mesh.stl
- link right_thumb_pp: geometry collision mesh filename=meshes/urdf/right/collision/right_collision_thumb_pp_mesh.s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; visual mesh filename=meshes/urdf/right/visual/right_visual_thumb_pp_mesh.stl
- link right_tower: geometry collision mesh filename=meshes/urdf/right/collision/right_collision_tower_hull_mesh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; collision mesh filename=meshes/urdf/right/collision/right_collision_tower_main_mesh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
