Commit message: baoding optimized for shadowlite

File: roto/assets/shadow_lite/sr_hand_touchlab.urdf (robot description, URDF)
Before this commit: robot shadowhand_motor, 26 links, 25 joints
Links:
- link rh_ffdistal: geometry collision mesh filename=meshes/touchlab/fingertip_v5_simple.stl scale=0.1 0.1 0.1; visual mesh filename=meshes/touchlab/fingertip_v5_simple.stl scale=0.1 0.1 0.1
- link rh_mfdistal: geometry collision mesh filename=meshes/touchlab/fingertip_v5_simple.stl scale=0.1 0.1 0.1; visual mesh filename=meshes/touchlab/fingertip_v5_simple.stl scale=0.1 0.1 0.1
- link rh_rfdistal: geometry collision mesh filename=meshes/touchlab/fingertip_v5_simple.stl scale=0.1 0.1 0.1; visual mesh filename=meshes/touchlab/fingertip_v5_simple.stl scale=0.1 0.1 0.1
- link rh_thdistal: geometry collision mesh filename=meshes/touchlab/fingertip_v5_simple.stl scale=0.1 0.1 0.1; visual mesh filename=meshes/touchlab/fingertip_v5_simple.stl scale=0.1 0.1 0.1
Joints:
- joint rh_FFJ1: mimic joint=rh_FFJ2 multiplier=1.0 offset=0.0 -> (none)
- joint rh_MFJ1: mimic joint=rh_MFJ2 multiplier=1.0 offset=0.0 -> (none)
- joint rh_RFJ1: mimic joint=rh_RFJ2 multiplier=1.0 offset=0.0 -> (none)
- joint rh_THJ1: origin xyz=0 0 0.032 rpy=0 0 0 -> xyz=0 0 0.034 rpy=0 0 0

Commit message: shadowlite works with 55gm balls - fixed fingertips mismatch

File: roto/assets/shadow_lite/sr_hand_touchlab.urdf (robot description, URDF)
Before this commit: robot shadowhand_motor, 26 links, 25 joints
Joints:
- joint rh_FFJ2: limit lower=0 upper=1.5707963267948966 effort=2 velocity=2.0 -> lower=0 upper=1.63 effort=2 velocity=2.0
- joint rh_MFJ2: limit lower=0 upper=1.5707963267948966 effort=2 velocity=2.0 -> lower=0 upper=1.63 effort=2 velocity=2.0
- joint rh_RFJ2: limit lower=0 upper=1.5707963267948966 effort=2 velocity=2.0 -> lower=0 upper=1.63 effort=2 velocity=2.0
