Commit message: sysid: coupled-finger gating, actuator tuning + sim-vs-hw diagnostics
Coupling/mimic work:
- roto_env: optional measured-J2 gate for J1 (couple_gate_j1_on_measured /
  couple_gate_lo_frac) so the J1 mimic can't lead its J2 driver
- shadowlite cfg: gate flags

Sys-id / tuning tooling (scripts/):
- test_coupling.py: verify J2 commanded/reaching its limit, J1 early-firing,
  runtime stiffness/damping/effort override
- tune_grip.py: sweep coupled-joint gains for ball grip/lift (1 ball, mass/
  diameter knobs, clean deterministic test: friction DR/noise/terminations off)
- test_gate_fraction.py, view_coupling.py, plot_mimic_check.py

Sim-vs-hardware comparison tooling (scripts/):
- record_tactile_sim.py, plot_tactile_compare.py
- replay_traj_hw.py (command / sim_pos replay), plot_traj_compare.py
- my_policy_node.py: tactile logging + 80->4 taxel aggregation

Assets: regenerated shadow_lite USDs (meshcol variant), config/urdf updates.

Co-Authored-By: Claude Opus 4.8 <noreply@anthropic.com>

File: roto/assets/shadow_lite/sr_hand_touchlab.urdf (robot description, URDF)
Before this commit: robot shadowhand_motor, 26 links, 25 joints
Joints:
- joint rh_FFJ1: limit lower=0 upper=1.5707963267948966 effort=2 velocity=2.0 -> lower=0 upper=1.396 effort=2 velocity=2.0
- joint rh_FFJ2: limit lower=0 upper=1.63 effort=2 velocity=2.0 -> lower=0 upper=1.745 effort=2 velocity=2.0
- joint rh_MFJ1: limit lower=0 upper=1.5707963267948966 effort=2 velocity=2.0 -> lower=0 upper=1.396 effort=2 velocity=2.0
- joint rh_MFJ2: limit lower=0 upper=1.63 effort=2 velocity=2.0 -> lower=0 upper=1.745 effort=2 velocity=2.0
- joint rh_RFJ1: limit lower=0 upper=1.5707963267948966 effort=2 velocity=2.0 -> lower=0 upper=1.396 effort=2 velocity=2.0
- joint rh_RFJ2: limit lower=0 upper=1.63 effort=2 velocity=2.0 -> lower=0 upper=1.745 effort=2 velocity=2.0
