Commit message: Stateful backlash coupling, DR, settle phase, viewer + diagnostics, USD asset
- roto_env: stateful J1<-J2 backlash coupling (strict curl, early-unlock uncurl
  at per-episode R, freeze-until-R reversal), latched-direction J2 selection,
  ball-settle state freeze.
- shadowlite: coupling cfg flags, per-episode unlock-R DR, hand tilt fixed at 15°.
- baoding: ball-settle phase.
- shadow_hand_lite + assets: prebuilt USD/URDF + STL meshes.
- scripts: coupling slider viewer, backlash/robustness/self-contact diagnostics.

File: roto/assets/shadow_lite/SHADOW_TOUCHLAB.urdf (robot description, URDF)
Before this commit: robot shadowhand_motor, 26 links, 25 joints
Links:
- link rh_ffdistal: geometry collision mesh filename=meshes/touchlab/fingertip_v5_simple_m.stl scale=1.0 1.0 1.0; visual mesh filename=meshes/touchlab/fingertip_v5_simple_m.stl scale=1.0 1.0 1.0
- link rh_ffknuckle: geometry collision mesh filename=meshes/components/f_knuckle/f_knuckle_G1M5_m.stl scale=1.0 1.0 1.0; visual mesh filename=meshes/components/f_knuckle/f_knuckle_G1M5_m.stl scale=1.0 1.0 1.0
- link rh_ffmiddle: geometry collision mesh filename=meshes/components/f_middle/f_middle_G1M5_m.stl scale=1.0 1.0 1.0; visual mesh filename=meshes/components/f_middle/f_middle_G1M5_m.stl scale=1.0 1.0 1.0
- link rh_ffproximal: geometry collision mesh filename=meshes/components/f_proximal/f_proximal_G1M5_m.stl scale=1.0 1.0 1.0; visual mesh filename=meshes/components/f_proximal/f_proximal_G1M5_m.stl scale=1.0 1.0 1.0
- link rh_forearm: geometry collision mesh filename=meshes/components/forearm/forearm_G1M5.stl scale=1.0 1.0 1.0; visual mesh filename=meshes/components/forearm/forearm_G1M5.stl scale=1.0 1.0 1.0
- link rh_mfdistal: geometry collision mesh filename=meshes/touchlab/fingertip_v5_simple_m.stl scale=1.0 1.0 1.0; visual mesh filename=meshes/touchlab/fingertip_v5_simple_m.stl scale=1.0 1.0 1.0
- link rh_mfknuckle: geometry collision mesh filename=meshes/components/f_knuckle/f_knuckle_G1M5_m.stl scale=1.0 1.0 1.0; visual mesh filename=meshes/components/f_knuckle/f_knuckle_G1M5_m.stl scale=1.0 1.0 1.0
- link rh_mfmiddle: geometry collision mesh filename=meshes/components/f_middle/f_middle_G1M5_m.stl scale=1.0 1.0 1.0; visual mesh filename=meshes/components/f_middle/f_middle_G1M5_m.stl scale=1.0 1.0 1.0
- link rh_mfproximal: geometry collision mesh filename=meshes/components/f_proximal/f_proximal_G1M5_m.stl scale=1.0 1.0 1.0; visual mesh filename=meshes/components/f_proximal/f_proximal_G1M5_m.stl scale=1.0 1.0 1.0
- link rh_palm: geometry collision mesh filename=meshes/components/palm/palm_G1M5_m.stl scale=1.0 1.0 1.0; visual mesh filename=meshes/components/palm/palm_G1M5_m.stl scale=1.0 1.0 1.0
- link rh_rfdistal: geometry collision mesh filename=meshes/touchlab/fingertip_v5_simple_m.stl scale=1.0 1.0 1.0; visual mesh filename=meshes/touchlab/fingertip_v5_simple_m.stl scale=1.0 1.0 1.0
- link rh_rfknuckle: geometry collision mesh filename=meshes/components/f_knuckle/f_knuckle_G1M5_m.stl scale=1.0 1.0 1.0; visual mesh filename=meshes/components/f_knuckle/f_knuckle_G1M5_m.stl scale=1.0 1.0 1.0
- link rh_rfmiddle: geometry collision mesh filename=meshes/components/f_middle/f_middle_G1M5_m.stl scale=1.0 1.0 1.0; visual mesh filename=meshes/components/f_middle/f_middle_G1M5_m.stl scale=1.0 1.0 1.0
- link rh_rfproximal: geometry collision mesh filename=meshes/components/f_proximal/f_proximal_G1M5_m.stl scale=1.0 1.0 1.0; visual mesh filename=meshes/components/f_proximal/f_proximal_G1M5_m.stl scale=1.0 1.0 1.0
- link rh_thdistal: geometry collision mesh filename=meshes/touchlab/fingertip_v5_simple_m.stl scale=1.0 1.0 1.0; visual mesh filename=meshes/touchlab/fingertip_v5_simple_m.stl scale=1.0 1.0 1.0
- link rh_thmiddle: geometry collision mesh filename=meshes/components/th_middle/th_middle_G1M5_m.stl scale=1.0 1.0 1.0; visual mesh filename=meshes/components/th_middle/th_middle_G1M5_m.stl scale=1.0 1.0 1.0
- link rh_thproximal: geometry collision mesh filename=meshes/components/th_proximal/th_proximal_G1M5_m.stl scale=1.0 1.0 1.0; visual mesh filename=meshes/components/th_proximal/th_proximal_G1M5_m.stl scale=1.0 1.0 1.0

File: roto/assets/shadow_lite/sr_hand_touchlab.urdf (robot description, URDF)
Before this commit: robot shadowhand_motor, 26 links, 25 joints
Links:
- link rh_thproximal: geometry collision cylinder length=0.018 radius=0.012; visual mesh filename=meshes/components/th_proximal/th_proximal_G1M5.stl scale=0.001 0.001 0.001

File: roto/assets/shadow_lite/sr_hand_touchlab_visual.urdf (robot description, URDF)
Before this commit: robot shadowhand_motor, 26 links, 25 joints
Links:
- link rh_ffdistal: geometry visual mesh filename=meshes/touchlab/fingertip_v5_simple_m.stl scale=1.0 1.0 1.0
- link rh_ffknuckle: geometry visual mesh filename=meshes/components/f_knuckle/f_knuckle_G1M5_m.stl scale=1.0 1.0 1.0
- link rh_ffmiddle: geometry visual mesh filename=meshes/components/f_middle/f_middle_G1M5_m.stl scale=1.0 1.0 1.0
- link rh_ffproximal: geometry visual mesh filename=meshes/components/f_proximal/f_proximal_G1M5_m.stl scale=1.0 1.0 1.0
- link rh_forearm: geometry visual mesh filename=meshes/components/forearm/forearm_G1M5.stl scale=1.0 1.0 1.0
- link rh_mfdistal: geometry visual mesh filename=meshes/touchlab/fingertip_v5_simple_m.stl scale=1.0 1.0 1.0
- link rh_mfknuckle: geometry visual mesh filename=meshes/components/f_knuckle/f_knuckle_G1M5_m.stl scale=1.0 1.0 1.0
- link rh_mfmiddle: geometry visual mesh filename=meshes/components/f_middle/f_middle_G1M5_m.stl scale=1.0 1.0 1.0
- link rh_mfproximal: geometry visual mesh filename=meshes/components/f_proximal/f_proximal_G1M5_m.stl scale=1.0 1.0 1.0
- link rh_palm: geometry visual mesh filename=meshes/components/palm/palm_G1M5_m.stl scale=1.0 1.0 1.0
- link rh_rfdistal: geometry visual mesh filename=meshes/touchlab/fingertip_v5_simple_m.stl scale=1.0 1.0 1.0
- link rh_rfknuckle: geometry visual mesh filename=meshes/components/f_knuckle/f_knuckle_G1M5_m.stl scale=1.0 1.0 1.0
- link rh_rfmiddle: geometry visual mesh filename=meshes/components/f_middle/f_middle_G1M5_m.stl scale=1.0 1.0 1.0
- link rh_rfproximal: geometry visual mesh filename=meshes/components/f_proximal/f_proximal_G1M5_m.stl scale=1.0 1.0 1.0
- link rh_thbase: geometry visual box size=0.001 0.001 0.001
- link rh_thdistal: geometry visual mesh filename=meshes/touchlab/fingertip_v5_simple_m.stl scale=1.0 1.0 1.0
- link rh_thhub: geometry visual box size=0.001 0.001 0.001
- link rh_thmiddle: geometry visual mesh filename=meshes/components/th_middle/th_middle_G1M5_m.stl scale=1.0 1.0 1.0
- link rh_thproximal: geometry visual mesh filename=meshes/components/th_proximal/th_proximal_G1M5_m.stl scale=1.0 1.0 1.0
